File: D1MiniRFM95.brd (EAGLE design)
At the start: 25.4 x 33 mm, 5 parts

Commit message: v4.01
Parts:
- removed JP1: Sensor, adafruit:1X03-CLEANBIG
- added ANT: (no value), adafruit:1X1-BIGPOGO
- added C1: (no value), resistor:C025-024X044
- added D3: (no value), jumper:JP1
- moved LORA 2.79 mm to (20.6, 6.60)
Connections:
- new net D3B: D3.2, LORA.P$16
- net 3.3V: now also C1.1; no longer JP1.1
- net ANT: now also ANT.P$1
- net D3: now also D3.1; no longer LORA.P$16
- net D4: no longer JP1.3
- net D5: now also LORA.P$4
- net D6: now also LORA.P$2
- net D7: now also LORA.P$3
- net GND: now also C1.2; no longer JP1.2
Routing:
- net D4: track 35.8 -> 0.00 mm
- net D3B: track 0.00 -> 30.5 mm
- net D5: track 0.00 -> 18.8 mm
- net D6: track 0.00 -> 15.5 mm, vias 0 -> 1
- net D7: track 0.00 -> 15.0 mm
- net D8: track 18.4 -> 31.0 mm, vias 0 -> 1
- net D3: track 22.5 -> 16.9 mm
- net 3.3V: track 37.4 -> 33.6 mm
- net D0: track 28.5 -> 25.4 mm
- net ANT: track 11.8 -> 8.98 mm
- net D1: track 20.5 -> 17.7 mm
- net D2: track 21.2 -> 19.3 mm
Other:
- board text added: "D1 Mini RFM95 Shield v4"
- board text removed: "D1 Mini RFM95 Shield AM Kuipers"
