File: D1MiniRFM95.sch (EAGLE design)
At the start: 5 parts

Commit message: v4.01
Parts:
- removed JP1: Sensor, adafruit:PINHD-1X3CB
- added ANT: (no value), adafruit:PINHD-1X1-BIGPOGO
- added C1: (no value), resistor:C-EU025-024X044
- added D3: (no value), jumper:JP1Q
Connections:
- new net D3B: D3.2, LORA.DIO2
- net 3.3V: now also C1.1; no longer JP1.1
- net ANT: now also ANT.1
- net D3: now also D3.1; no longer LORA.DIO2
- net D4: no longer JP1.3
- net D5: now also LORA.SCK
- net D6: now also LORA.MISO
- net D7: now also LORA.MOSI
- net GND: now also C1.2; no longer JP1.2
Other:
- note added: "D1 mini"
- note added: "DRAFT - UNTESTED"
- note removed: "SKU: D1MSHO"
- note removed: "V1.1 (2016-03-08)"
